File: pcb/manufoldv2.kicad_sch (KiCad schematic)
At the start: 0 parts

Commit message: initial matrix setup
Parts:
- added J? (x2): Conn_02x05_Top_Bottom, symbol Connector_Generic:Conn_02x05_Top_Bottom
- added U1: ProMicro, symbol keebio:ProMicro
Connections:
- new net GND: J?.5 (Pin_5), J?.5 (Pin_5), U1.23 (GND), U1.3 (GND), U1.4 (GND)
- new net VCC: J?.1 (Pin_1), J?.1 (Pin_1), U1.21 (VCC), U1.24 (RAW)
- new net led: U1.13 (10/PB6)
- new net main_col1: J?.6 (Pin_6), U1.19 (A2/PF5)
- new net main_col2: J?.7 (Pin_7), U1.18 (A1/PF6)
- new net main_col3: J?.8 (Pin_8), U1.17 (A0/PF7)
- new net main_col4: U1.16 (15/PB1)
- new net main_col5: J?.9 (Pin_9), U1.15 (14/PB3)
- new net main_col6: J?.10 (Pin_10), U1.14 (16/PB2)
- new net main_led_neg: J?.2 (Pin_2)
- new net main_row1: U1.10 (7/PE6), U1.11 (8/PB4), U1.12 (9/PB5), U1.7 (4/PD4), U1.8 (5/PC6), U1.9 (6/PD7)
- new net main_row5: J?.3 (Pin_3)
- new net main_row6: J?.4 (Pin_4)
- new net reset: U1.22 (RST)
- new net scl: U1.6 (3/PD0)
- new net sda: U1.5 (2/PD1)
- new net serial: U1.2 (RX1/PD2)
- new net sub_col1: J?.6 (Pin_6)
- new net sub_col2: J?.7 (Pin_7)
- new net sub_col3: J?.8 (Pin_8)
- new net sub_col5: J?.9 (Pin_9)
- new net sub_col6: J?.10 (Pin_10)
- new net sub_led_neg: J?.2 (Pin_2)
- new net sub_row5: J?.3 (Pin_3)
- new net sub_row6: J?.4 (Pin_4)
- no-connect marks 0 -> 2
Other:
- added sheet Main Matrix (main.kicad_sch)
- added sheet Sub Matrix (sub.kicad_sch)
- title: (none) -> Manufold v2 Main Sheet
