File: pcb/manufoldv2.kicad_sch (KiCad schematic)
At the start: 3 parts, among them U1 ProMicro

Commit message: initial schematic
Parts:
- added J3: Conn_01x04_Female, symbol Connector:Conn_01x04_Female
- added J4: TRRS, symbol keebio:TRRS
- added JP1, JP2, JP3, JP4, JP5, JP6, JP7, JP8: SolderJumper_2_Open, symbol Jumper:SolderJumper_2_Open
- added Q1: Q_NMOS_GSD, symbol Device:Q_NMOS_GSD
- added R1, R2, R3: R, symbol Device:R
- gave numbers to parts that had none: 2
Connections:
- net GND: now also J4.1 (SLEEVE), JP4.1 (A), JP8.2 (B), Q1.2 (S); no longer J2.5 (Pin_5)
- net VCC: now also J4.3 (RING1), JP3.1 (A), JP7.2 (B), R2.1, R3.1; no longer J2.1 (Pin_1)
- net led: now also R1.1
- net main_led_neg: now also Q1.3 (D)
- net main_row1: no longer U1.10 (7/PE6), U1.11 (8/PB4), U1.12 (9/PB5), U1.8 (5/PC6), U1.9 (6/PD7)
- net main_row5: now also U1.11 (8/PB4)
- net main_row6: now also U1.12 (9/PB5)
- net scl: now also JP2.1 (A), JP6.2 (B), R3.2
- net sda: now also JP1.1 (A), JP5.2 (B), R2.2
- net serial: now also J4.2 (TIP)
- new net: J3.1 (Pin_1), JP4.2 (B), JP5.1 (A)
- new net: J3.2 (Pin_2), JP3.2 (B), JP6.1 (A)
- new net: J3.3 (Pin_3), JP2.2 (B), JP7.1 (A)
- new net: J3.4 (Pin_4), JP1.2 (B), JP8.1 (A)
- new net: Q1.1 (G), R1.2
- new net GND1: J2.5 (Pin_5)
- new net main_row2: U1.8 (5/PC6)
- new net main_row3: U1.9 (6/PD7)
- new net main_row4: U1.10 (7/PE6)
- new net sub_led_pos: J2.1 (Pin_1)
- no-connect marks 2 -> 3
Other:
- added sheet Mechanical (mech.kicad_sch)
- moved on the sheet: J1, J2

Commit message: add dual promicro footprint, associate footprints
Parts:
- added SW1: SW_Push, Jumper:SolderJumper-2_P1.3mm_Open_RoundedPad1.0x1.5mm, symbol Switch:SW_Push
- J1: footprint (none) -> Connector_PinHeader_1.27mm:PinHeader_2x05_P1.27mm_Horizontal
- J2: footprint (none) -> Connector_PinSocket_1.27mm:PinSocket_2x05_P1.27mm_Vertical
- J3: footprint (none) -> Connector_PinSocket_2.54mm:PinSocket_1x04_P2.54mm_Vertical
- J4: footprint (none) -> keebio:TRRS-PJ-320A-dual
- JP1, JP2, JP3, JP4, JP5, JP6, JP7, JP8: footprint (none) -> Jumper:SolderJumper-2_P1.3mm_Open_RoundedPad1.0x1.5mm
- Q1: footprint (none) -> keebio:SOT-23_Handsoldering
- R1, R2, R3: footprint (none) -> keebio:Resistor-Hybrid
- U1: footprint (none) -> promicro_dual:promicro_dual
Connections:
- net GND: now also SW1.2
- net reset: now also SW1.1

Commit message: initial routing
Parts:
- R1, R2, R3: footprint keebio:Resistor-Hybrid -> Resistor_SMD:R_0805_2012Metric
Changed lines of the file:
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@@
     (rev "A")
   )
+  (junction (at 64.77 129.54) (diameter 0) (color 0 0 0 0))
+  (junction (at 67.31 137.16) (diameter 0) (color 0 0 0 0))
+  (junction (at 86.36 40.64) (diameter 0) (color 0 0 0 0))
   (junction (at 43.18 48.26) (diameter 0) (color 0 0 0 0))
-  (junction (at 86.36 40.64) (diameter 0) (color 0 0 0 0))
-  (junction (at 64.77 129.54) (diameter 0) (color 0 0 0 0))
+  (junction (at 59.69 139.7) (diameter 0) (color 0 0 0 0))
   (junction (at 62.23 132.08) (diameter 0) (color 0 0 0 0))
-  (junction (at 59.69 139.7) (diameter 0) (color 0 0 0 0))
-  (junction (at 67.31 137.16) (diameter 0) (color 0 0 0 0))
   (no_connect (at 138.43 58.42))
+  (no_connect (at 81.28 50.8))
   (no_connect (at 45.72 40.64))
-  (no_connect (at 81.28 50.8))
   (wire (pts (xy 40.64 50.8) (xy 45.72 50.8))
     (stroke (width 0) (type default) (color 0 0 0 0))
@@
     (stroke (width 0) (type default) (color 0 0 0 0))
   )
+  (wire (pts (xy 86.36 38.1) (xy 86.36 40.64))
+    (stroke (width 0) (type default) (color 0 0 0 0))
+  )
   (wire (pts (xy 86.36 40.64) (xy 86.36 48.26))
     (stroke (width 0) (type default) (color 0 0 0 0))
   )
-  (wire (pts (xy 86.36 38.1) (xy 86.36 40.64))
-    (stroke (width 0) (type default) (color 0 0 0 0))
-  )
   (wire (pts (xy 33.02 124.46) (xy 43.18 124.46))
     (stroke (width 0) (type default) (color 0 0 0 0))
@@
     (stroke (width 0) (type default) (color 0 0 0 0))
   )
+  (wire (pts (xy 50.8 132.08) (xy 62.23 132.08))
+    (stroke (width 0) (type default) (color 0 0 0 0))
+  )
   (wire (pts (xy 62.23 132.08) (xy 62.23 147.32))
     (stroke (width 0) (type default) (color 0 0 0 0))
   )
-  (wire (pts (xy 50.8 132.08) (xy 62.23 132.08))
-    (stroke (width 0) (type default) (color 0 0 0 0))
-  )
   (wire (pts (xy 81.28 58.42) (xy 88.9 58.42))
     (stroke (width 0) (type default) (color 0 0 0 0))
@@
     (stroke (width 0) (type default) (color 0 0 0 0))
   )
+  (wire (pts (xy 62.23 121.92) (xy 62.23 132.08))
+    (stroke (width 0) (type default) (color 0 0 0 0))
+  )
   (wire (pts (xy 76.2 121.92) (xy 62.23 121.92))
     (stroke (width 0) (type default) (color 0 0 0 0))
   )
-  (wire (pts (xy 62.23 121.92) (xy 62.23 132.08))
-    (stroke (width 0) (type default) (color 0 0 0 0))
-  )
   (wire (pts (xy 186.69 43.1014) (xy 186.69 45.6414))
     (stroke (width 0) (type default) (color 0 0 0 0))
@@
     (stroke (width 0) (type default) (color 0 0 0 0))
   )
+  (wire (pts (xy 127 55.88) (xy 138.43 55.88))
+    (stroke (width 0) (type default) (color 0 0 0 0))
+  )
   (wire (pts (xy 127 50.8) (xy 127 55.88))
     (stroke (width 0) (type default) (color 0 0 0 0))
   )
-  (wire (pts (xy 127 55.88) (xy 138.43 55.88))
-    (stroke (width 0) (type default) (color 0 0 0 0))
-  )
   (wire (pts (xy 64.77 129.54) (xy 64.77 147.32))
     (stroke (width 0) (type default) (color 0 0 0 0))
@@
     (stroke (width 0) (type default) (color 0 0 0 0))
   )
+  (wire (pts (xy 50.8 116.84) (xy 67.31 116.84))
+    (stroke (width 0) (type default) (color 0 0 0 0))
+  )
   (wire (pts (xy 67.31 116.84) (xy 67.31 137.16))
     (stroke (width 0) (type default) (color 0 0 0 0))
   )
-  (wire (pts (xy 50.8 116.84) (xy 67.31 116.84))
-    (stroke (width 0) (type default) (color 0 0 0 0))
-  )
   (wire (pts (xy 67.31 137.16) (xy 67.31 147.32))
     (stroke (width 0) (type default) (color 0 0 0 0))
   )
+  (wire (pts (xy 59.69 139.7) (xy 50.8 139.7))
+    (stroke (width 0) (type default) (color 0 0 0 0))
+  )
   (wire (pts (xy 59.69 147.32) (xy 59.69 139.7))
     (stroke (width 0) (type default) (color 0 0 0 0))
   )
-  (wire (pts (xy 59.69 139.7) (xy 50.8 139.7))
-    (stroke (width 0) (type default) (color 0 0 0 0))
-  )
   (wire (pts (xy 33.02 116.84) (xy 43.18 116.84))
     (stroke (width 0) (type default) (color 0 0 0 0))
@@
     (stroke (width 0) (type default) (color 0 0 0 0))
   )
+  (wire (pts (xy 81.28 43.18) (xy 83.82 43.18))
+    (stroke (width 0) (type default) (color 0 0 0 0))
+  )
   (wire (pts (xy 83.82 43.18) (xy 83.82 71.12))
     (stroke (width 0) (type default) (color 0 0 0 0))
   )
-  (wire (pts (xy 81.28 43.18) (xy 83.82 43.18))
-    (stroke (width 0) (type default) (color 0 0 0 0))
-  )
   (wire (pts (xy 43.18 45.72) (xy 45.72 45.72))
     (stroke (width 0) (type default) (color 0 0 0 0))
   )
+  (wire (pts (xy 43.18 48.26) (xy 43.18 45.72))
+    (stroke (width 0) (type default) (color 0 0 0 0))
+  )
   (wire (pts (xy 43.18 71.12) (xy 43.18 48.26))
-    (stroke (width 0) (type default) (color 0 0 0 0))
-  )
-  (wire (pts (xy 43.18 48.26) (xy 43.18 45.72))
     (stroke (width 0) (type default) (color 0 0 0 0))
   )
@@
       (effects (font (size 1.27 1.27)) (justify left))
     )
-    (property "Footprint" "keebio:Resistor-Hybrid" (id 2) (at 47.752 157.48 90)
+    (property "Footprint" "Resistor_SMD:R_0805_2012Metric" (id 2) (at 47.752 157.48 90)
       (effects (font (size 1.27 1.27)) hide)
     )
@@
     (property "Reference" "R1" (id 0) (at 140.97 91.5375 90))
     (property "Value" "R" (id 1) (at 140.97 94.3126 90))
-    (property "Footprint" "keebio:Resistor-Hybrid" (id 2) (at 140.97 98.298 90)
+    (property "Footprint" "Resistor_SMD:R_0805_2012Metric" (id 2) (at 140.97 98.298 90)
       (effects (font (size 1.27 1.27)) hide)
     )
@@
       (effects (font (size 1.27 1.27)) (justify left))
     )
-    (property "Footprint" "keebio:Resistor-Hybrid" (id 2) (at 35.052 157.48 90)
+    (property "Footprint" "Resistor_SMD:R_0805_2012Metric" (id 2) (at 35.052 157.48 90)
       (effects (font (size 1.27 1.27)) hide)
     )
@@
     )
     (path "/d4ee606e-622a-4a74-b47d-0c32f3790916"
-      (reference "R1") (unit 1) (value "R") (footprint "keebio:Resistor-Hybrid")
+      (reference "R1") (unit 1) (value "R") (footprint "Resistor_SMD:R_0805_2012Metric")
     )
     (path "/d8aacc00-f895-40d9-9233-f599c1910ea2"
-      (reference "R2") (unit 1) (value "R") (footprint "keebio:Resistor-Hybrid")
+      (reference "R2") (unit 1) (value "R") (footprint "Resistor_SMD:R_0805_2012Metric")
     )
     (path "/6d3b3958-7327-4ee0-8610-96fdc33da4fc"
-      (reference "R3") (unit 1) (value "R") (footprint "keebio:Resistor-Hybrid")
+      (reference "R3") (unit 1) (value "R") (footprint "Resistor_SMD:R_0805_2012Metric")
     )
     (path "/1bc1b30e-956e-440e-95f5-f165eca705b0/f8f282b6-a577-4253-9f4f-77c63b247060"
