File: pcb/main.kicad_sch (KiCad schematic)
At the start: 104 parts

Commit message: initial schematic
Parts:
- gave numbers to parts that had none: 78

Commit message: add dual promicro footprint, associate footprints
Parts:
- D11, D12, D13, D14, D15, D16, D21, D22, D23, D24, D25, D26, D31, D32, D33, D34, D35, D36, D41, D42, D43, D44, D45, D46, D53, D54: footprint (none) -> keebio:Diode-dual
- R11, R12, R13, R14, R15, R16, R21, R22, R23, R24, R25, R26, R31, R32, R33, R34, R35, R36, R41, R42, R43, R44, R45, R46, R53, R54: footprint (none) -> keebio:Resistor-Hybrid
- SW11, SW12, SW13, SW14, SW15, SW16, SW21, SW22, SW23, SW24, SW25, SW26, SW31, SW32, SW33, SW34, SW35, SW36, SW41, SW42, SW43, SW44, SW45, SW46, SW53, SW54: footprint (none) -> keebio:Triple-Dual-1u-LED

Commit message: initial routing
Connections:
- net main_col5: no longer SW16.1, SW26.1, SW36.1, SW46.1
- net main_row1: no longer D21.1 (K), D22.1 (K), D23.1 (K), D24.1 (K), D25.1 (K), D26.1 (K), D31.1 (K), D32.1 (K), D33.1 (K), D34.1 (K), D35.1 (K), D36.1 (K), D41.1 (K), D42.1 (K), D43.1 (K), D44.1 (K), D45.1 (K), D46.1 (K), D53.1 (K), D54.1 (K)
- net main_led renamed main_led_neg
- new net main_col6: SW16.1, SW26.1, SW36.1, SW46.1
- new net main_row2: D21.1 (K), D22.1 (K), D23.1 (K), D24.1 (K), D25.1 (K), D26.1 (K)
- new net main_row3: D31.1 (K), D32.1 (K), D33.1 (K), D34.1 (K), D35.1 (K), D36.1 (K)
- new net main_row4: D41.1 (K), D42.1 (K), D43.1 (K), D44.1 (K), D45.1 (K), D46.1 (K)
- new net main_row5: D53.1 (K), D54.1 (K)
