File: pcb/sub.kicad_sch (KiCad schematic)
At the start: 23 parts

Commit message: initial schematic
Parts:
- gave numbers to parts that had none: 19
Connections:
- net sub_col5: no longer SW56.1
- net sub_col6: now also SW56.1
- net VCC renamed sub_led_pos
- net sub_led renamed sub_led_neg

Commit message: add dual promicro footprint, associate footprints
Parts:
- D51, D52, D55, D56: footprint (none) -> keebio:Diode-dual
- D61, D62, D63, D65, D66: footprint (none) -> keebio:D_SOD123F
- R51, R52, R55, R56: footprint (none) -> keebio:Resistor-Hybrid
- SN1, SN2: footprint digikey-footprints:Switch_Nav_12.4x12.4mm_SMD_JS5208 -> digikey:Switch_Nav_12.4x12.4mm_SMD_JS5208
- SW51, SW52, SW55, SW56: footprint (none) -> keebio:Triple-Dual-1u-LED
Changed lines of the file:
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@@
     (rev "A")
   )
-  (junction (at 76.2 50.8) (diameter 0) (color 0 0 0 0))
+  (junction (at 198.12 68.58) (diameter 0) (color 0 0 0 0))
+  (junction (at 181.61 68.58) (diameter 0) (color 0 0 0 0))
+  (junction (at 152.4 120.5049) (diameter 0) (color 0 0 0 0))
+  (junction (at 63.5 68.58) (diameter 0) (color 0 0 0 0))
+  (junction (at 63.5 50.8) (diameter 0) (color 0 0 0 0))
+  (junction (at 88.9 68.58) (diameter 0) (color 0 0 0 0))
+  (junction (at 144.78 115.4249) (diameter 0) (color 0 0 0 0))
+  (junction (at 160.02 125.5849) (diameter 0) (color 0 0 0 0))
   (junction (at 116.84 120.5049) (diameter 0) (color 0 0 0 0))
   (junction (at 109.22 125.5849) (diameter 0) (color 0 0 0 0))
   (junction (at 88.9 50.8) (diameter 0) (color 0 0 0 0))
+  (junction (at 165.1 68.58) (diameter 0) (color 0 0 0 0))
+  (junction (at 76.2 68.58) (diameter 0) (color 0 0 0 0))
+  (junction (at 76.2 50.8) (diameter 0) (color 0 0 0 0))
   (junction (at 119.38 115.4249) (diameter 0) (color 0 0 0 0))
-  (junction (at 160.02 125.5849) (diameter 0) (color 0 0 0 0))
-  (junction (at 152.4 120.5049) (diameter 0) (color 0 0 0 0))
-  (junction (at 181.61 68.58) (diameter 0) (color 0 0 0 0))
-  (junction (at 198.12 68.58) (diameter 0) (color 0 0 0 0))
-  (junction (at 63.5 50.8) (diameter 0) (color 0 0 0 0))
-  (junction (at 76.2 68.58) (diameter 0) (color 0 0 0 0))
-  (junction (at 144.78 115.4249) (diameter 0) (color 0 0 0 0))
-  (junction (at 165.1 68.58) (diameter 0) (color 0 0 0 0))
-  (junction (at 63.5 68.58) (diameter 0) (color 0 0 0 0))
-  (junction (at 88.9 68.58) (diameter 0) (color 0 0 0 0))
   (wire (pts (xy 88.9 66.04) (xy 88.9 68.58))
     (stroke (width 0) (type default) (color 0 0 0 0))
@@
     (stroke (width 0) (type default) (color 0 0 0 0))
   )
+  (wire (pts (xy 152.4 142.0949) (xy 152.4 120.5049))
+    (stroke (width 0) (type default) (color 0 0 0 0))
+  )
   (wire (pts (xy 142.24 142.0949) (xy 152.4 142.0949))
     (stroke (width 0) (type default) (color 0 0 0 0))
   )
-  (wire (pts (xy 152.4 142.0949) (xy 152.4 120.5049))
-    (stroke (width 0) (type default) (color 0 0 0 0))
-  )
   (wire (pts (xy 109.22 147.1749) (xy 109.22 125.5849))
     (stroke (width 0) (type default) (color 0 0 0 0))
@@
     (stroke (width 0) (type default) (color 0 0 0 0))
   )
+  (wire (pts (xy 142.24 120.5049) (xy 152.4 120.5049))
+    (stroke (width 0) (type default) (color 0 0 0 0))
+  )
   (wire (pts (xy 152.4 112.8849) (xy 152.4 120.5049))
     (stroke (width 0) (type default) (color 0 0 0 0))
   )
-  (wire (pts (xy 142.24 120.5049) (xy 152.4 120.5049))
-    (stroke (width 0) (type default) (color 0 0 0 0))
-  )
   (wire (pts (xy 106.68 115.4249) (xy 119.38 115.4249))
     (stroke (width 0) (type default) (color 0 0 0 0))
@@
     (stroke (width 0) (type default) (color 0 0 0 0))
   )
+  (wire (pts (xy 116.84 112.8849) (xy 116.84 120.5049))
+    (stroke (width 0) (type default) (color 0 0 0 0))
+  )
   (wire (pts (xy 116.84 120.5049) (xy 121.92 120.5049))
     (stroke (width 0) (type default) (color 0 0 0 0))
   )
-  (wire (pts (xy 116.84 112.8849) (xy 116.84 120.5049))
-    (stroke (width 0) (type default) (color 0 0 0 0))
-  )
   (wire (pts (xy 144.78 102.7249) (xy 144.78 105.2649))
     (stroke (width 0) (type default) (color 0 0 0 0))
@@
     (stroke (width 0) (type default) (color 0 0 0 0))
   )
+  (wire (pts (xy 160.02 125.5849) (xy 142.24 125.5849))
+    (stroke (width 0) (type default) (color 0 0 0 0))
+  )
   (wire (pts (xy 160.02 112.8849) (xy 160.02 125.5849))
-    (stroke (width 0) (type default) (color 0 0 0 0))
-  )
-  (wire (pts (xy 160.02 125.5849) (xy 142.24 125.5849))
     (stroke (width 0) (type default) (color 0 0 0 0))
   )
@@
       (effects (font (size 1.27 1.27)) (justify right))
     )
-    (property "Footprint" "" (id 2) (at 165.1 64.77 0)
+    (property "Footprint" "keebio:Diode-dual" (id 2) (at 165.1 64.77 0)
       (effects (font (size 1.27 1.27)) hide)
     )
@@
       (effects (font (size 1.27 1.27)) (justify left))
     )
-    (property "Footprint" "" (id 2) (at 88.9 62.23 0)
+    (property "Footprint" "keebio:Triple-Dual-1u-LED" (id 2) (at 88.9 62.23 0)
       (effects (font (size 1.27 1.27)) hide)
     )
@@
       (effects (font (size 1.524 1.524)))
     )
-    (property "Footprint" "digikey-footprints:Switch_Nav_12.4x12.4mm_SMD_JS5208" (id 2) (at 137.16 115.4249 0)
+    (property "Footprint" "digikey:Switch_Nav_12.4x12.4mm_SMD_JS5208" (id 2) (at 137.16 115.4249 0)
       (effects (font (size 1.524 1.524)) (justify left) hide)
     )
@@
       (effects (font (size 1.27 1.27)) (justify right))
     )
-    (property "Footprint" "" (id 2) (at 181.61 64.77 0)
+    (property "Footprint" "keebio:Diode-dual" (id 2) (at 181.61 64.77 0)
       (effects (font (size 1.27 1.27)) hide)
     )
@@
       (effects (font (size 1.27 1.27)) (justify right))
     )
-    (property "Footprint" "" (id 2) (at 198.12 64.77 0)
+    (property "Footprint" "keebio:Diode-dual" (id 2) (at 198.12 64.77 0)
       (effects (font (size 1.27 1.27)) hide)
     )
@@
       (effects (font (size 1.27 1.27)) (justify right))
     )
-    (property "Footprint" "" (id 2) (at 144.78 109.0749 0)
+    (property "Footprint" "keebio:D_SOD123F" (id 2) (at 144.78 109.0749 0)
       (effects (font (size 1.27 1.27)) hide)
     )
@@
       (effects (font (size 1.27 1.27)) (justify left))
     )
-    (property "Footprint" "" (id 2) (at 63.5 62.23 0)
+    (property "Footprint" "keebio:Triple-Dual-1u-LED" (id 2) (at 63.5 62.23 0)
       (effects (font (size 1.27 1.27)) hide)
     )
@@
       (effects (font (size 1.27 1.27)) (justify left))
     )
-    (property "Footprint" "" (id 2) (at 87.122 54.61 90)
+    (property "Footprint" "keebio:Resistor-Hybrid" (id 2) (at 87.122 54.61 90)
       (effects (font (size 1.27 1.27)) hide)
     )
@@
       (effects (font (size 1.27 1.27)) (justify left))
     )
-    (property "Footprint" "" (id 2) (at 165.1 55.88 0)
+    (property "Footprint" "keebio:Triple-Dual-1u-LED" (id 2) (at 165.1 55.88 0)
       (effects (font (size 1.27 1.27)) hide)
     )
@@
       (effects (font (size 1.27 1.27)) (justify left))
     )
-    (property "Footprint" "" (id 2) (at 50.8 62.23 0)
+    (property "Footprint" "keebio:Triple-Dual-1u-LED" (id 2) (at 50.8 62.23 0)
       (effects (font (size 1.27 1.27)) hide)
     )
@@
       (effects (font (size 1.27 1.27)) (justify left))
     )
-    (property "Footprint" "" (id 2) (at 74.422 54.61 90)
+    (property "Footprint" "keebio:Resistor-Hybrid" (id 2) (at 74.422 54.61 90)
       (effects (font (size 1.27 1.27)) hide)
     )
@@
       (effects (font (size 1.27 1.27)) (justify right))
     )
-    (property "Footprint" "" (id 2) (at 109.22 109.0749 0)
+    (property "Footprint" "keebio:D_SOD123F" (id 2) (at 109.22 109.0749 0)
       (effects (font (size 1.27 1.27)) hide)
     )
@@
       (effects (font (size 1.27 1.27)) (justify left))
     )
-    (property "Footprint" "" (id 2) (at 214.63 55.88 0)
+    (property "Footprint" "keebio:Triple-Dual-1u-LED" (id 2) (at 214.63 55.88 0)
       (effects (font (size 1.27 1.27)) hide)
     )
@@
       (effects (font (size 1.27 1.27)) (justify right))
     )
-    (property "Footprint" "" (id 2) (at 214.63 64.77 0)
+    (property "Footprint" "keebio:Diode-dual" (id 2) (at 214.63 64.77 0)
       (effects (font (size 1.27 1.27)) hide)
     )
@@
       (effects (font (size 1.27 1.27)) (justify right))
     )
-    (property "Footprint" "" (id 2) (at 160.02 109.0749 0)
+    (property "Footprint" "keebio:D_SOD123F" (id 2) (at 160.02 109.0749 0)
       (effects (font (size 1.27 1.27)) hide)
     )
@@
       (effects (font (size 1.27 1.27)) (justify left))
     )
-    (property "Footprint" "" (id 2) (at 181.61 55.88 0)
+    (property "Footprint" "keebio:Triple-Dual-1u-LED" (id 2) (at 181.61 55.88 0)
       (effects (font (size 1.27 1.27)) hide)
     )
@@
       (effects (font (size 1.27 1.27)) (justify left))
     )
-    (property "Footprint" "" (id 2) (at 198.12 55.88 0)
+    (property "Footprint" "keebio:Triple-Dual-1u-LED" (id 2) (at 198.12 55.88 0)
       (effects (font (size 1.27 1.27)) hide)
     )
@@
       (effects (font (size 1.27 1.27)) (justify left))
     )
-    (property "Footprint" "" (id 2) (at 61.722 54.61 90)
+    (property "Footprint" "keebio:Resistor-Hybrid" (id 2) (at 61.722 54.61 90)
       (effects (font (size 1.27 1.27)) hide)
     )
@@
       (effects (font (size 1.27 1.27)) (justify right))
     )
-    (property "Footprint" "" (id 2) (at 152.4 109.0749 0)
+    (property "Footprint" "keebio:D_SOD123F" (id 2) (at 152.4 109.0749 0)
       (effects (font (size 1.27 1.27)) hide)
     )
@@
       (effects (font (size 1.27 1.27)) (justify right))
     )
-    (property "Footprint" "" (id 2) (at 116.84 109.0749 0)
+    (property "Footprint" "keebio:D_SOD123F" (id 2) (at 116.84 109.0749 0)
       (effects (font (size 1.27 1.27)) hide)
     )
@@
       (effects (font (size 1.27 1.27)) (justify left))
     )
-    (property "Footprint" "" (id 2) (at 76.2 62.23 0)
+    (property "Footprint" "keebio:Triple-Dual-1u-LED" (id 2) (at 76.2 62.23 0)
       (effects (font (size 1.27 1.27)) hide)
     )
@@
       (effects (font (size 1.27 1.27)) (justify left))
     )
-    (property "Footprint" "" (id 2) (at 49.022 54.61 90)
+    (property "Footprint" "keebio:Resistor-Hybrid" (id 2) (at 49.022 54.61 90)
       (effects (font (size 1.27 1.27)) hide)
     )
@@
       (effects (font (size 1.524 1.524)))
     )
-    (property "Footprint" "digikey-footprints:Switch_Nav_12.4x12.4mm_SMD_JS5208" (id 2) (at 137.16 137.0149 0)
-      (effects (font (size 1.524 1.524)) (justify left) hide)
-    )
+    (property "Footprint" "digikey:Switch_Nav_12.4x12.4mm_SMD_JS5208" (id 2) (at 137.16 137.0149 0)
+      (effects (font (size 1.524 1.524)) (justify left) hide)
+    )

Commit message: initial routing
Connections:
- net sub_row1 renamed sub_row5
- net sub_row2 renamed sub_row6
Changed lines of the file:
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@@
     (rev "A")
   )
+  (junction (at 63.5 50.8) (diameter 0) (color 0 0 0 0))
   (junction (at 198.12 68.58) (diameter 0) (color 0 0 0 0))
+  (junction (at 119.38 115.4249) (diameter 0) (color 0 0 0 0))
+  (junction (at 109.22 125.5849) (diameter 0) (color 0 0 0 0))
   (junction (at 181.61 68.58) (diameter 0) (color 0 0 0 0))
+  (junction (at 116.84 120.5049) (diameter 0) (color 0 0 0 0))
+  (junction (at 63.5 68.58) (diameter 0) (color 0 0 0 0))
+  (junction (at 88.9 68.58) (diameter 0) (color 0 0 0 0))
+  (junction (at 76.2 68.58) (diameter 0) (color 0 0 0 0))
   (junction (at 152.4 120.5049) (diameter 0) (color 0 0 0 0))
-  (junction (at 63.5 68.58) (diameter 0) (color 0 0 0 0))
-  (junction (at 63.5 50.8) (diameter 0) (color 0 0 0 0))
-  (junction (at 88.9 68.58) (diameter 0) (color 0 0 0 0))
   (junction (at 144.78 115.4249) (diameter 0) (color 0 0 0 0))
+  (junction (at 165.1 68.58) (diameter 0) (color 0 0 0 0))
+  (junction (at 76.2 50.8) (diameter 0) (color 0 0 0 0))
   (junction (at 160.02 125.5849) (diameter 0) (color 0 0 0 0))
-  (junction (at 116.84 120.5049) (diameter 0) (color 0 0 0 0))
-  (junction (at 109.22 125.5849) (diameter 0) (color 0 0 0 0))
   (junction (at 88.9 50.8) (diameter 0) (color 0 0 0 0))
-  (junction (at 165.1 68.58) (diameter 0) (color 0 0 0 0))
-  (junction (at 76.2 68.58) (diameter 0) (color 0 0 0 0))
-  (junction (at 76.2 50.8) (diameter 0) (color 0 0 0 0))
-  (junction (at 119.38 115.4249) (diameter 0) (color 0 0 0 0))
   (wire (pts (xy 88.9 66.04) (xy 88.9 68.58))
     (stroke (width 0) (type default) (color 0 0 0 0))
@@
     (stroke (width 0) (type default) (color 0 0 0 0))
   )
+  (wire (pts (xy 142.24 142.0949) (xy 152.4 142.0949))
+    (stroke (width 0) (type default) (color 0 0 0 0))
+  )
   (wire (pts (xy 152.4 142.0949) (xy 152.4 120.5049))
     (stroke (width 0) (type default) (color 0 0 0 0))
   )
-  (wire (pts (xy 142.24 142.0949) (xy 152.4 142.0949))
-    (stroke (width 0) (type default) (color 0 0 0 0))
-  )
   (wire (pts (xy 109.22 147.1749) (xy 109.22 125.5849))
     (stroke (width 0) (type default) (color 0 0 0 0))
@@
     (stroke (width 0) (type default) (color 0 0 0 0))
   )
+  (wire (pts (xy 152.4 112.8849) (xy 152.4 120.5049))
+    (stroke (width 0) (type default) (color 0 0 0 0))
+  )
   (wire (pts (xy 142.24 120.5049) (xy 152.4 120.5049))
     (stroke (width 0) (type default) (color 0 0 0 0))
   )
-  (wire (pts (xy 152.4 112.8849) (xy 152.4 120.5049))
-    (stroke (width 0) (type default) (color 0 0 0 0))
-  )
   (wire (pts (xy 106.68 115.4249) (xy 119.38 115.4249))
     (stroke (width 0) (type default) (color 0 0 0 0))
@@
     (stroke (width 0) (type default) (color 0 0 0 0))
   )
+  (wire (pts (xy 160.02 112.8849) (xy 160.02 125.5849))
+    (stroke (width 0) (type default) (color 0 0 0 0))
+  )
   (wire (pts (xy 160.02 125.5849) (xy 142.24 125.5849))
     (stroke (width 0) (type default) (color 0 0 0 0))
   )
-  (wire (pts (xy 160.02 112.8849) (xy 160.02 125.5849))
-    (stroke (width 0) (type default) (color 0 0 0 0))
-  )
-  (global_label "sub_row1" (shape passive) (at 158.75 68.58 180) (fields_autoplaced)
+  (global_label "sub_row5" (shape passive) (at 158.75 68.58 180) (fields_autoplaced)
     (effects (font (size 1.27 1.27)) (justify right))
     (property "Intersheet References" "${INTERSHEET_REFS}" (id 0) (at 147.5679 68.5006 0)
@@
     )
   )
-  (global_label "sub_row2" (shape passive) (at 106.68 115.4249 180) (fields_autoplaced)
+  (global_label "sub_row6" (shape passive) (at 106.68 115.4249 180) (fields_autoplaced)
     (effects (font (size 1.27 1.27)) (justify right))
     (property "Intersheet References" "${INTERSHEET_REFS}" (id 0) (at 95.4979 115.3455 0)
